File: carte principal.kicad_pcb (KiCad board)
At the start: 2 copper layers, 60 x 25 mm, 31 parts, among them J1 UART CL, J10 I2C Extension, J2 UART CM, J3 UART CC, J4 UART CE, J5 con AX12A, J6 connecteur puissance, J9 I2C Extension, U1 XIAO-ESP32-S3-DIP

Commit message: apdavph
Parts:
- D4, R11: moved to F.Cu
- moved R11 6.09 mm to (211.9, 77.5), turned to 180 degrees
- moved R7 3.88 mm to (210.5, 82.2), turned to 0 degrees
- moved D4 2.75 mm to (211.9, 79.8), turned to 180 degrees
- moved D2 1.60 mm to (215.5, 82.2), turned to 180 degrees
Routing:
- net +12V: track 25.7 -> 35.5 mm
- net U8: track 18.9 -> 23.8 mm
- net U6: track 7.41 -> 10.0 mm
- net U4: track 28.8 -> 26.8 mm
- net +3.3V: track 61.6 -> 60.3 mm
- net U3: track 28.9 -> 28.0 mm
- net LI AX12A: track 24.3 -> 25.1 mm, vias 1 -> 0
- net +5V: track 51.2 -> 52.0 mm
- net Net-(D2-A): track 2.56 -> 2.05 mm
- net GND: vias 1 -> 6
