File: carte principal.kicad_sch (KiCad schematic)
At the start: 28 parts, among them J1 UART CL, J10 I2C Extension, J2 UART CM, J3 UART CC, J5 con AX12A, J6 connecteur puissance, J9 I2C Extension, U1 XIAO-ESP32-S3-DIP

Commit message: first routage
Parts:
- added J4: UART CE, Connector_Molex:Molex_KK-254_AE-6410-03A_1x03_P2.54mm_Vertical, symbol Connector_Generic:Conn_01x03
- added R12, R13: 47, Resistor_SMD:R_1206_3216Metric_Pad1.30x1.75mm_HandSolder, symbol Device:R
- U1: footprint Module:MOUDLE14P-XIAO-DIP-SMD -> Seeed Studio XIAO Series Library:XIAO-ESP32S3-DIP
Connections:
- net GND: now also J4.3 (Pin_3)
- net at U1.7 (U0TXD/D6/TX): now also R13.2
- net at U1.8 (U0RXD/D7/RX): now also R12.1
- new net U7: J4.1 (Pin_1), R13.1
- new net U8: J4.2 (Pin_2), R12.2
Other:
- moved on the sheet: J2, J3, J5

Commit message: fix
Parts:
- removed J6: connecteur puissance, Connector_Molex:Molex_KK-254_AE-6410-04A_1x04_P2.54mm_Vertical, symbol Connector_Generic:Conn_01x04
- added J12: conn 24v, Connector_AMASS:AMASS_XT60-F_1x02_P7.20mm_Vertical, symbol Connector_Generic:Conn_01x02
- added J7: conn 3.3v, Connector_AMASS:AMASS_XT30U-F_1x02_P5.0mm_Vertical, symbol Connector_Generic:Conn_01x02
- added J8: conn 5v, Connector_Molex:Molex_KK-254_AE-6410-02A_1x02_P2.54mm_Vertical, symbol Connector_Generic:Conn_01x02
Connections:
- net +3.3V: now also J7.2 (Pin_2)
- net +5V: now also J8.1 (Pin_1)
- net GND: now also J12.1 (Pin_1), J7.1 (Pin_1), J8.2 (Pin_2)
- new net +24V: J12.2 (Pin_2)
